File: hushlog.kicad_sch (KiCad schematic)
At the start: 0 parts

Commit message: Add README with schematic image
Parts:
- added C1, C11, C17, C18: 1uF, symbol Device:C
- added C10: 10uF, symbol Device:C
- added C12, C13, C14, C2, C3, C4, C5, C6, C7, C8, C9: 100nF, symbol Device:C
- added C15, C16: 15pF, symbol Device:C
- added J1: USB_C_Receptacle_USB2.0_16P, symbol Connector:USB_C_Receptacle_USB2.0_16P
- added J2: SWD, symbol Connector_Generic:Conn_01x03
- added R1, R2: 5.1k, symbol Device:R
- added R3, R6: 10k, symbol Device:R
- added R4, R5: 1k, symbol Device:R
- added R7, R8: 27R, symbol Device:R
- added SW1: BOOTSEL, symbol Switch:SW_Push
- added SW2: RESET, symbol Switch:SW_Push
- added U1: RP2040, Package_DFN_QFN:QFN-56-1EP_7x7mm_P0.4mm_EP3.2x3.2mm, symbol MCU_RaspberryPi:RP2040
- added U2: W25Q128JVS, Package_SO:SOIC-8_5.23x5.23mm_P1.27mm, symbol Memory_Flash:W25Q128JVS
- added U3: AP2112K-3.3, Package_TO_SOT_SMD:SOT-23-5, symbol Regulator_Linear:AP2112K-3.3
- added Y1: 12MHz, symbol Device:Crystal_GND24
Connections:
- new net: C16.1, R5.2, Y1.3
- new net: R4.2, SW1.1
- new net: J1.A5 (CC1), R1.1
- new net: J1.B5 (CC2), R2.1
- new net +1V1: C11.1, C12.1, C13.1, U1.23 (DVDD), U1.45 (VREG_VOUT), U1.50 (DVDD)
- new net +3.3V: C1.1, C10.1, C14.1, C18.1, C2.1, C3.1, C4.1, C5.1, C6.1, C7.1, C8.1, C9.1, R3.1, R6.1, U1.1 (IOVDD), U1.10 (IOVDD), U1.22 (IOVDD), U1.33 (IOVDD), U1.42 (IOVDD), U1.43 (ADC_AVDD), U1.44 (VREG_VIN), U1.48 (USB_VDD), U1.49 (IOVDD), U2.8 (VCC), U3.5 (VOUT)
- new net GND: C1.2, C10.2, C11.2, C12.2, C13.2, C14.2, C15.2, C16.2, C17.2, C18.2, C2.2, C3.2, C4.2, C5.2, C6.2, C7.2, C8.2, C9.2, J1.A1 (GND), J1.A12 (GND), J1.B1 (GND), J1.B12 (GND), J1.S1 (SHIELD), J2.2 (Pin_2), R1.2, R2.2, SW1.2, SW2.2, U1.19 (TESTEN), U1.57 (GND), U2.4 (GND), U3.2 (GND), Y1.2, Y1.4
- new net QSPI_SCLK: U1.52 (QSPI_SCLK), U2.6 (CLK)
- new net QSPI_SD0: U1.53 (QSPI_SD0), U2.5 (DI(IO0))
- new net QSPI_SD1: U1.55 (QSPI_SD1), U2.2 (DO(IO1))
- new net QSPI_SD2: U1.54 (QSPI_SD2), U2.3 (IO2)
- new net QSPI_SD3: U1.51 (QSPI_SD3), U2.7 (IO3)
- new net QSPI_SS: R3.2, R4.1, U1.56 (~{QSPI_SS}), U2.1 (~{CS})
- new net RUN: R6.2, SW2.1, U1.26 (RUN)
- new net SWCLK: J2.1 (Pin_1), U1.24 (SWCLK)
- new net SWDIO: J2.3 (Pin_3), U1.25 (SWDIO)
- new net USB_CONN_D+: J1.A6 (D+), J1.B6 (D+), R8.1
- new net USB_CONN_D-: J1.A7 (D-), J1.B7 (D-), R7.1
- new net USB_D+: R8.2, U1.47 (USB_DP)
- new net USB_D-: R7.2, U1.46 (USB_DM)
- new net VBUS: C17.1, J1.A4 (VBUS), J1.A9 (VBUS), J1.B4 (VBUS), J1.B9 (VBUS), U3.1 (VIN), U3.3 (EN)
- new net XIN: C15.1, U1.20 (XIN), Y1.1
- new net XOUT: R5.1, U1.21 (XOUT)
- no-connect marks 0 -> 2
Other:
- note added: "12 MHz crystal, e.g. ABM8-272-T3 (CL = 10 pF). C15/C16 = 2 x (CL - ~3 pF stray). Recalculate C15/C16 if you pick a different crystal. R5 limits drive level."
- note added: "1V1 core, from the internal regulator: C11: at pin 45 (VREG_VOUT) C12, C13: at DVDD pins 23 and 50"
- note added: "3V3 decoupling - where each cap goes on the PCB: C1: at pin 44 (VREG_VIN) C2-C7: one per IOVDD pin (1, 10, 22, 33, 42, 49) C8: at pin 48 (USB_VDD) C9: at pin 43 (ADC_AVDD) C10: bulk, anywhere on 3V3"
- note added: "3V3 rail from USB VBUS (5 V). AP2112K-3.3: 600 mA, needs 1 uF in and out (C17, C18)."
- note added: "QSPI flash. The RP2040 has no internal flash, it boots from U2. Hold SW1 (BOOTSEL) while applying power to enter the USB bootloader. R3 is optional."
- note added: "SW2 resets the MCU (RUN low). J2 is the debug port: 1 = SWCLK, 2 = GND, 3 = SWDIO."
- note added: "USB 2.0 device. R1/R2 (5.1k to GND) tell a USB-C host to supply 5 V. R7/R8: place close to U1 pins 46/47. Route D+/D- as a 90 ohm diff pair. No ESD protection or VBUS fuse yet - add before a production spin."

Commit message: Add ADS1220 analog front end
Parts:
- added C19, C22, C25, C26: 100nF, symbol Device:C
- added C20, C21, C23, C24: 10nF, symbol Device:C
- added C27, C28: 1uF, symbol Device:C
- added J3: IN_A, symbol Connector:Screw_Terminal_01x02
- added J4: IN_B, symbol Connector:Screw_Terminal_01x02
- added J5: GND, symbol Connector:Screw_Terminal_01x02
- added R10, R11, R12, R9: 1k, symbol Device:R
- added U4: ADS1220IPW, Package_SO:TSSOP-16_4.4x5mm_P0.65mm, symbol Analog_ADC:ADS1220xPW
- added U5: TPS7A2033PDBV, Package_TO_SOT_SMD:SOT-23-5, symbol Regulator_Linear:TPS7A2033PDBV
- U2: footprint Package_SO:SOIC-8_5.23x5.23mm_P1.27mm -> Package_SO:SOIC-8_3.9x4.9mm_P1.27mm
Connections:
- net +3.3V: now also C25.1, U4.13 (DVDD)
- net GND: now also C20.1, C21.2, C23.1, C24.2, C25.2, C26.2, C27.2, C28.2, J5.1 (Pin_1), J5.2 (Pin_2), U4.3 (CLK), U4.4 (DGND), U4.5 (AVSS), U5.2 (GND)
- net VBUS: now also C27.1, U5.1 (IN), U5.3 (EN)
- net ADC_SCLK: now reaches U1.4 (GPIO2)
- net ADC_SCLK: now also U4.1 (SCLK)
- net ADC_MOSI: now reaches U1.5 (GPIO3)
- net ADC_MOSI: now also U4.16 (DIN)
- net ADC_MISO: now reaches U1.6 (GPIO4)
- net ADC_MISO: now also U4.15 (DOUT/~{DRDY})
- net ADC_CS: now reaches U1.7 (GPIO5)
- net ADC_CS: now also U4.2 (~{CS})
- net ADC_DRDY: now reaches U1.8 (GPIO6)
- net ADC_DRDY: now also U4.14 (~{DRDY})
- new net: J4.2 (Pin_2), R12.1
- new net: J3.1 (Pin_1), R9.1
- new net: J4.1 (Pin_1), R11.1
- new net: J3.2 (Pin_2), R10.1
- new net +3.3VA: C26.1, C28.1, U4.12 (AVDD), U5.5 (OUT)
- new net AIN0: C19.1, C20.2, R9.2, U4.11 (AIN0/REFP1)
- new net AIN1: C19.2, C21.1, R10.2, U4.10 (AIN1)
- new net AIN2: C22.1, C23.2, R11.2, U4.7 (AIN2)
- new net AIN3: C22.2, C24.1, R12.2, U4.6 (AIN3/REFN1)
- no-connect marks 2 -> 4
Other:
- note added: "ANALOG FRONT END - ADS1220 24-bit ADC, two differential pairs (or four single-ended inputs), own low-noise supply"
- note added: "Analog supply: TPS7A2033 (7 uVrms) fed straight from VBUS, so AVDD never touches the digital +3.3V rail. Layout: C26 right at U4 pin 12 (AVDD), C25 right at pin 13 (DVDD). Keep U5 and its caps next to the ADC."
- note added: "Input filter per pair: 1k in each leg, 100nF across the pair, 10nF from each leg to GND (differential fc ~760 Hz, common-mode fc ~16 kHz). Differential: sensor on pin 1 (+) and pin 2 (-), PGA gain up to 128. Single-ended: sensor from AINx to the GND terminal, PGA bypassed, gain 1-4. A floating source (bare thermocouple) needs a DC path: bias its - leg, e.g. link pin 2 to GND and bypass the PGA, o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"
- note added: "SPI0, mode 1 (CPOL=0, CPHA=1): GPIO2 SCLK, GPIO3 MOSI, GPIO4 MISO, GPIO5 CS, GPIO6 DRDY (falling edge = data ready). CLK tied to GND = internal oscillator. REFP0/REFN0 unused (internal 2.048 V reference); they may float per the datasheet."
